File: CommandeJF.kicad_pcb (KiCad board)
At the start: 2 copper layers, 100 x 70 mm, 14 parts, among them J1 Conn_01x02, J2 Conn_01x02, J3 Conn_01x04, K1 RelaisSRD, T1 Trou, T2 Trou, T3 Trou, T4 Trou, U101 MP1584, U2 DS3231

Commit message: Mise en forme
Parts:
- TR1: value Transistor_TO92 -> 2N2222A
- XA101: value Arduino_Pro_Mini -> Arduino_Mini
- moved D2 2.30 mm to (160.0, 86.2)
Connections:
- J1 pad 1: +24V -> GND1
- J1 pad 2: Net-(J1-Pad2) -> +24V
- U101 pad 1: +24V -> GND1
- U101 pad 2: Net-(J1-Pad2) -> +24V
Routing:
- net Net-(J1-Pad2): track 14.3 -> 0.00 mm
- net GND1: track 0.00 -> 13.5 mm
- net Net-(D2-Pad2): track 22.9 -> 33.7 mm
- net SDA: track 170.8 -> 161.0 mm
- net SCL: track 111.7 -> 107.7 mm
- net GND: track 127.7 -> 125.1 mm
- net +5V: track 255.6 -> 255.0 mm
- net +24V: track 13.7 -> 14.3 mm
Other:
- net class 24V: trace_width 1 -> 2
- board text added: "24V"
- board text added: "5V"
- board text added: "GND"
- board text added: "IN"
- board text added: "OUT"
- board text added: "SCL"
- board text added: "SDA"

Commit message: Arduino nano
Parts:
- removed U2: DS3231, Timer_RTC:RTC_DS3231
- removed XA101: Arduino_Mini, Arduino:Arduino_Pro_Mini
- added R101: R1.2k, Resistance:R_025W, F.Cu at (154.1, 84.7)
- added U1: DS3231, Timer_RTC:RTC_DS3231, F.Cu at (115.1, 94.2)
- added XA1: Arduino_Nano_Socket, Arduino:Arduino_Nano_Module_sur_Socket, F.Cu at (142.5, 106.9)
- C101: value CP -> CP47µF; footprint capacitors:CP_5x11mm -> capacitors:CP_5x11mm_hor
- J1: value Conn_01x02 -> Conn_01x04; footprint TerminalBlock_Phoenix:TerminalBlock_Phoenix_MKDS-1,5-2-5.08_1x02_P5.08mm_Horizontal -> TerminalBlock_Phoenix:TerminalBlock_Phoenix_MKDS-1,5-4-5.08_1x04_P5.08mm_Horizontal
- moved C101 9.14 mm to (177.9, 110.1)
- moved J1 4.70 mm to (107.7, 63.8)
- moved TR1 2.60 mm to (155.3, 69.6), turned to 180 degrees
Connections:
- C101 pad 1: +5V -> +12V
- D2 pad 1: +5V -> +12V
- J1 pad 2: +24V -> Net-(J1-Pad2)
- J3 pad 1: SCL -> GND
- J3 pad 2: SDA -> +5V
- J3 pad 3: +5V -> SCL
- J3 pad 4: GND -> SDA
- K1 pad A1: +5V -> +12V
- TR1 pad 1: GND -> Net-(D2-Pad2)
- TR1 pad 2: SIG -> Net-(R101-Pad1)
- TR1 pad 3: Net-(D2-Pad2) -> GND
- U101 pad 4: +5V -> +12V
Routing:
- net +12V: track 0.00 -> 173.7 mm
- net +5V: track 255.0 -> 92.5 mm
- net SDA: track 161.0 -> 64.8 mm
- net SCL: track 107.7 -> 71.7 mm
- net SIG: track 30.4 -> 9.71 mm
- net GND: track 125.1 -> 140.4 mm
- net Net-(R101-Pad1): track 0.00 -> 8.01 mm
- net Net-(J1-Pad2): track 0.00 -> 5.08 mm
- net +24V: track 14.3 -> 10.5 mm
- net GND1: track 13.5 -> 10.5 mm
Other:
- net class 12V added: clearance 0.2, trace_width 1, via_dia 0.8, via_drill 0.4
- board text added: "0"
- board text added: "24"
- board text removed: "24V"

Commit message: version 1
Parts:
- removed C101: CP47µF, capacitors:CP_5x11mm_hor
- D2: value Diode_1N4148 -> 1N4148
- K1: value RelaisSRD -> Relais
- R101: value R1.2k -> R1k
- TR1: value 2N2222A -> Transistor_TO92
- moved D2 23.5 mm to (170.7, 65.3)
- moved T1 22.4 mm to (110.0, 40.0)
- moved T2 22.4 mm to (200.0, 40.0)
- moved XA1 19.5 mm to (153.2, 90.6)
- moved J1 19.5 mm to (118.4, 47.5)
- moved U1 19.5 mm to (125.8, 77.9)
- moved U101 19.5 mm to (137.7, 55.1)
- moved J2 19.5 mm to (187.7, 55.5)
- moved J3 19.5 mm to (131.2, 95.4)
- moved K1 19.5 mm to (177.2, 67.7)
- moved T4 18.4 mm to (200.7, 105.0)
- moved T3 18.0 mm to (110.0, 105.0)
- moved R101 16.7 mm to (159.7, 69.0)
- moved TR1 16.3 mm to (158.4, 53.6), turned to 0 degrees
Connections:
- TR1 pad 1: Net-(D2-Pad2) -> GND
- TR1 pad 3: GND -> Net-(D2-Pad2)
- XA1 pad D11: (no net) -> SIG
- XA1 pad D9: SIG -> (no net)
Routing:
- net GND: track 140.4 -> 0.00 mm
- net +12V: track 173.7 -> 97.7 mm
- net Net-(R101-Pad1): track 8.01 -> 12.3 mm
- net SIG: track 9.71 -> 9.10 mm
- added copper zone on B.Cu, net GND
Other:
- board size 100 x 70 mm -> 100 x 75 mm
- net class 12V: trace_width 1 -> 1.5
- net class Default: trace_width 0.8 -> 1

Commit message: Version finale
Parts:
- XA1: value Arduino_Nano_Socket -> Arduino_Nano
- moved J1 1.10 mm to (118.4, 46.4)
Connections:
- J2 pad 2: Net-(J2-Pad2) -> Net-(J2-Pad1)
- K1 pad 11: Net-(J2-Pad2) -> +24V
Routing:
- net +24V: track 10.5 -> 113.3 mm
- net Net-(J2-Pad2): track 27.5 -> 0.00 mm
- net Net-(J2-Pad1): track 21.9 -> 26.9 mm
Other:
- board text added: "0V"
- board text added: "24V"
- board text added: "Afficheur"
- board text added: "Interrupteur jours fériés"
- board text added: "ON"
- board text removed: "0"
- board text removed: "24"
- board text removed: "IN"
