File: CommandeJF.sch (KiCad schematic (older format))
At the start: 14 parts, among them J1 Conn_01x02, J2 Conn_01x02, J3 Conn_01x04, K1 RelaisSRD, T1 Trou, T2 Trou, T3 Trou, T4 Trou, U101 MP1584, U2 DS3231

Commit message: Mise en forme
Parts:
- TR1: value Transistor_TO92 -> 2N2222A
Connections:
- net +24V: now also J1.2 (Pin_2), U101.2 (+IN); no longer J1.1 (Pin_1), U101.1 (-IN)
- new net GND1: J1.1 (Pin_1), U101.1 (-IN)
Changed lines of the file:
@@
 $EndComp
 Wire Wire Line
-	2100 1650 2200 1650
-Wire Wire Line
-	2100 1900 2300 1900
+	2100 1900 2150 1900
 $Comp
 L power:+24V #PWR02
 U 1 1 639F9EC2
-P 2200 1650
-F 0 "#PWR02" H 2200 1500 50  0001 C CNN
-F 1 "+24V" H 2215 1823 50  0000 C CNN
-F 2 "" H 2200 1650 50  0001 C CNN
-F 3 "" H 2200 1650 50  0001 C CNN
-	1    2200 1650
-	1    0    0    -1
-$EndComp
-Connection ~ 2200 1650
-Wire Wire Line
-	2200 1650 2300 1650
+P 2150 1900
+F 0 "#PWR02" H 2150 1750 50  0001 C CNN
+F 1 "+24V" H 2165 2073 50  0000 C CNN
+F 2 "" H 2150 1900 50  0001 C CNN
+F 3 "" H 2150 1900 50  0001 C CNN
+	1    2150 1900
+	-1   0    0    1
+$EndComp
 $Comp
 L power:+5V #PWR03
@@
 P 7100 3650
 F 0 "TR1" H 7291 3696 50  0000 L CNN
-F 1 "Transistor_TO92" H 7291 3605 50  0000 L CNN
+F 1 "2N2222A" H 7291 3605 50  0000 L CNN
 F 2 "Transistor:TO-92" H 7300 3575 50  0001 L CIN
 F 3 "" H 7100 3650 50  0001 L CNN
@@
 Connection ~ 900  4650
 Connection ~ 900  4950
+Connection ~ 2150 1900
+Wire Wire Line
+	2150 1900 2300 1900
+Wire Wire Line
+	2100 1650 2150 1650
+$Comp
+L power:GND1 #PWR0108
+U 1 1 6426DB69
+P 2150 1650
+F 0 "#PWR0108" H 2150 1400 50  0001 C CNN
+F 1 "GND1" H 2155 1477 50  0000 C CNN
+F 2 "" H 2150 1650 50  0001 C CNN
+F 3 "" H 2150 1650 50  0001 C CNN
+	1    2150 1650
+	-1   0    0    1
+$EndComp
+Connection ~ 2150 1650
+Wire Wire Line
+	2150 1650 2300 1650
 $EndSCHEMATC

Commit message: Arduino nano
Parts:
- removed J1: Conn_01x02, TerminalBlock_Phoenix:TerminalBlock_Phoenix_MKDS-1,5-2-5.08_1x02_P5.08mm_Horizontal, symbol Connector_Generic:Conn_01x02
- removed U2: DS3231, Timer_RTC:RTC_DS3231, symbol Timer_RTC:DS3231
- removed XA101: Arduino_Pro_Mini, Arduino:Arduino_Pro_Mini, symbol Arduino:Arduino_Pro_Mini
- added J1: Conn_01x04, TerminalBlock_Phoenix:TerminalBlock_Phoenix_MKDS-1,5-4-5.08_1x04_P5.08mm_Horizontal, symbol Connector_Generic:Conn_01x04
- added R101: R1.2k, Resistance:R_025W, symbol Personnel:R
- added U1: DS3231, Timer_RTC:RTC_DS3231, symbol Timer_RTC:DS3231
- added XA1: Arduino_Nano_Socket, Arduino:Arduino_Nano_Module_sur_Socket, symbol Arduino:Arduino_Nano_Socket
- C101: value CP -> CP47µF; footprint capacitors:CP_5x11mm -> capacitors:CP_5x11mm_hor
Connections:
- net +24V: now also J1.4 (Pin_4)
- net +5V: now also J3.2 (Pin_2), U1.3 (VCC), XA1.5V; no longer C101.1, D2.1 (K), J3.3 (Pin_3), K1.A1, U101.4 (+OUT)
- net GND: now also J3.1 (Pin_1), U1.4 (GND), XA1.GND1 (GND); no longer J3.4 (Pin_4)
- net GND1: now also J1.1 (Pin_1)
- net SCL: now also J3.3 (Pin_3), U1.1 (SCL), XA1.A5 (A5_SCL); no longer J3.1 (Pin_1)
- net SDA: now also J3.4 (Pin_4), U1.2 (SDA), XA1.A4 (A4_SDA); no longer J3.2 (Pin_2)
- net SIG: now also R101.2, XA1.D9; no longer TR1.2 (B)
- new net: R101.1, TR1.2 (B)
- new net: J1.2 (Pin_2), J1.3 (Pin_3)
- new net +12V: C101.1, D2.1 (K), K1.A1, U101.4 (+OUT), XA1.VIN

Commit message: version 1
Parts:
- removed C101: CP47µF, capacitors:CP_5x11mm_hor, symbol Personnel:CP
- D2: value Diode_1N4148 -> 1N4148
- K1: value RelaisSRD -> Relais
- R101: value R1.2k -> R1k
- TR1: value 2N2222A -> Transistor_TO92
Connections:
- net SIG: now also XA1.D11 (D11_MOSI); no longer XA1.D9
Changed lines of the file:
@@
 $EndDescr
-$Comp
-L Personnel:Transistor_TO92 TR1
-U 1 1 63A006C4
-P 7100 3650
-F 0 "TR1" H 7291 3696 50  0000 L CNN
-F 1 "2N2222A" H 7291 3605 50  0000 L CNN
-F 2 "Transistor:TO-92" H 7300 3575 50  0001 L CIN
-F 3 "" H 7100 3650 50  0001 L CNN
-	1    7100 3650
-	1    0    0    -1
-$EndComp
 $Comp
 L Personnel:RelaisSRD K1
@@
 P 7400 2900
 F 0 "K1" H 7830 2946 50  0000 L CNN
-F 1 "RelaisSRD" H 7830 2855 50  0000 L CNN
+F 1 "Relais" H 7830 2855 50  0000 L CNN
 F 2 "Relay_THT:Relais_SRD" H 8670 2870 50  0001 C CNN
 F 3 "https://gfinder.findernet.com/public/attachments/36/EN/S36EN.pdf" H 7400 2900 50  0001 C CNN
@@
 Wire Wire Line
 	4200 6600 4650 6600
-Text GLabel 4350 3850 2    50   Input ~ 0
+Text GLabel 4350 4050 2    50   Input ~ 0
 SIG
 Text GLabel 6200 3650 0    50   Input ~ 0
@@
 P 6450 2850
 F 0 "D2" V 6450 2930 50  0000 L CNN
-F 1 "Diode_1N4148" H 6450 2750 50  0001 C CNN
+F 1 "1N4148" H 6450 2750 50  0001 C CNN
 F 2 "pth_diodes:diode_do35" H 6450 2675 50  0001 C CNN
 F 3 "" H 6450 2850 50  0001 C CNN
@@
 P 6500 3650
 F 0 "R101" V 6293 3650 50  0000 C CNN
-F 1 "R1.2k" V 6384 3650 50  0000 C CNN
+F 1 "R1k" V 6384 3650 50  0000 C CNN
 F 2 "Resistance:R_025W" V 6430 3650 50  0001 C CNN
 F 3 "~" H 6500 3650 50  0001 C CNN
@@
 Wire Wire Line
 	6200 3650 6350 3650
-$Comp
-L Personnel:CP C101
-U 1 1 642EAB77
-P 950 4800
-F 0 "C101" H 832 4754 50  0000 R CNN
-F 1 "CP47µF" H 832 4845 50  0000 R CNN
-F 2 "capacitors:CP_5x11mm_hor" H 988 4650 50  0001 C CNN
-F 3 "~" H 950 4800 50  0001 C CNN
-	1    950  4800
-	-1   0    0    1
-$EndComp
-Wire Wire Line
-	1550 4550 950  4550
-Wire Wire Line
-	950  4550 950  4650
-Connection ~ 1550 4550
-Wire Wire Line
-	950  4950 1750 4950
-Connection ~ 1750 4950
 $Comp
 L Connector_Generic:Conn_01x04 J1
@@
 Wire Wire Line
 	2200 1950 2300 1950
+$Comp
+L Personnel:Transistor_TO92 TR1
+U 1 1 642D8B0A
+P 7100 3650
+F 0 "TR1" H 7291 3696 50  0000 L CNN
+F 1 "Transistor_TO92" H 7291 3605 50  0000 L CNN
+F 2 "Transistor:TO-92" H 7300 3575 50  0001 L CIN
+F 3 "" H 7100 3650 50  0001 L CNN
+	1    7100 3650
+	1    0    0    -1
+$EndComp
 $EndSCHEMATC

Commit message: Version finale
Connections:
- net +24V: now also K1.11
- net at J2.2 (Pin_2): now also J2.1 (Pin_1), K1.14; no longer K1.11
Other:
- moved on the sheet: J2
Changed lines of the file:
@@
 L Connector_Generic:Conn_01x02 J2
 U 1 1 63A045DA
-P 8550 2800
-F 0 "J2" H 8630 2792 50  0000 L CNN
-F 1 "Conn_01x02" H 8630 2701 50  0000 L CNN
-F 2 "TerminalBlock_Phoenix:TerminalBlock_Phoenix_MKDS-1,5-2-5.08_1x02_P5.08mm_Horizontal" H 8550 2800 50  0001 C CNN
-F 3 "~" H 8550 2800 50  0001 C CNN
-	1    8550 2800
-	-1   0    0    -1
-$EndComp
-Wire Wire Line
-	8750 3200 7600 3200
+P 8200 2250
+F 0 "J2" H 8280 2242 50  0000 L CNN
+F 1 "Conn_01x02" H 8280 2151 50  0000 L CNN
+F 2 "TerminalBlock_Phoenix:TerminalBlock_Phoenix_MKDS-1,5-2-5.08_1x02_P5.08mm_Horizontal" H 8200 2250 50  0001 C CNN
+F 3 "~" H 8200 2250 50  0001 C CNN
+	1    8200 2250
+	1    0    0    1
+$EndComp
 $Comp
 L power:+5V #PWR07
@@
 $EndComp
 Wire Wire Line
-	8750 2800 8750 2500
-Wire Wire Line
-	8750 3200 8750 2900
-Wire Wire Line
 	3350 1650 3350 1600
 $Comp
@@
 	-1   0    0    1
 $EndComp
-Wire Wire Line
-	8750 2500 7700 2500
-Wire Wire Line
-	7700 2500 7700 2600
 Wire Wire Line
 	2150 1650 2300 1650
@@
 	1    0    0    -1
 $EndComp
+$Comp
+L power:+24V #PWR0112
+U 1 1 642FFB92
+P 7800 3300
+F 0 "#PWR0112" H 7800 3150 50  0001 C CNN
+F 1 "+24V" V 7815 3428 50  0000 L CNN
+F 2 "" H 7800 3300 50  0001 C CNN
+F 3 "" H 7800 3300 50  0001 C CNN
+	1    7800 3300
+	0    1    1    0
+$EndComp
+Wire Wire Line
+	7800 3300 7600 3300
+Wire Wire Line
+	7600 3300 7600 3200
+Wire Wire Line
+	8000 2250 7700 2250
+Wire Wire Line
+	7700 2250 7700 2600
+Wire Wire Line
+	8000 2150 8000 2250
+Connection ~ 8000 2250
 $EndSCHEMATC
